File: KiCad/ss_v2/ss_v2.kicad_pcb (KiCad board)
At the start: 2 copper layers, 59 parts, among them J1 PJ-313D-B-SMT, J2 UJC-HP-M-G-5-MSMT-TR, J3 DC-005-20A, J4 Conn_02x03_Top_Bottom, J5 Conn_02x03_Counter_Clockwise, J6 Conn_01x08_Pin, J7 Conn_01x04, Q1 BSN20, Q2 IRF7416TRPBF, Q3 BSN20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

Commit message: Erster Routing Versuch
Parts:
- U3: value TPS62125DSG -> TPS62175DQCR; footprint Package_SON:WSON-8-1EP_2x2mm_P0.5mm_EP0.9x1.6mm_ThermalVias -> TPS62175DQCR:DQC0010A
- moved U3 0.30 mm to (229.1, 76.8)
- turned R9 to 180 degrees
Connections:
- net Net-(J1-Pad2A) renamed output_power
- U3 pad 4: GND -> unconnected-(U3-NC-Pad4)
- U3 pad 6: +5V -> GND
- U3 pad 7: Net-(U3-SW) -> unconnected-(U3-PG-Pad7)
- U3 pad 9: GND -> Net-(U3-SW)
Routing:
- net +5V: track 0.00 -> 279.3 mm, vias 0 -> 9
- net +12V: track 0.00 -> 96.5 mm, vias 0 -> 1
- net reset: track 0.00 -> 48.5 mm
- net VBUS: track 0.00 -> 39.5 mm
- net sens: track 0.00 -> 26.9 mm
- net GND: track 0.00 -> 18.3 mm
- net cc1: track 0.00 -> 11.8 mm
- net cc2: track 0.00 -> 11.4 mm
- net Net-(R2-Pad1): track 0.00 -> 8.80 mm
- net Net-(U1-PB7): track 0.00 -> 8.11 mm
- net Net-(U1-PB6): track 0.00 -> 7.83 mm
- net Net-(U2-+): track 0.00 -> 7.67 mm
- net Net-(U2--): track 0.00 -> 6.92 mm
- net bl: track 0.00 -> 6.74 mm
- net Net-(U3-FB): track 0.00 -> 6.41 mm
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- added copper zone on F.Cu, net +12V
- added copper zone on F.Cu, net output_power
