File: KiCad/ss_v2/ss_v2.kicad_sch (KiCad schematic)
At the start: 57 parts, among them J1 PJ-313D-B-SMT, J2 UJC-HP-M-G-5-MSMT-TR, J3 DC-005-20A, J4 Conn_02x03_Top_Bottom, J5 Conn_02x03_Counter_Clockwise, J6 Conn_01x08_Pin, J7 Conn_01x04, Q1 BSN20, Q2 IRF7416TRPBF, Q3 BSN20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

Commit message: Standby pin hinzufeguegt
Parts:
- added R25, R26: 10k, Resistor_SMD:R_1206_3216Metric_Pad1.30x1.75mm_HandSolder, symbol Device:R
Connections:
- net +5V: now also R25.1
- net GND: now also R26.2
- net standby: now reaches U1.19 (ADC6)
- net standby: now also R25.2, R26.1
Changed lines of the file:
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@@
   (junction (at 116.84 108.585) (diameter 0) (color 0 0 0 0)
   )
+  (junction (at 90.17 177.165) (diameter 0) (color 0 0 0 0)
+  )
   (junction (at 152.4 36.195) (diameter 0) (color 0 0 0 0)
   )
@@
     (stroke (width 0) (type default))
   )
+  (wire (pts (xy 90.17 177.165) (xy 90.17 179.07))
+    (stroke (width 0) (type default))
+  )
   (wire (pts (xy 40.64 170.18) (xy 41.91 170.18))
     (stroke (width 0) (type default))
@@
     (stroke (width 0) (type default))
   )
+  (wire (pts (xy 90.17 175.26) (xy 90.17 177.165))
+    (stroke (width 0) (type default))
+  )
   (wire (pts (xy 19.685 63.5) (xy 28.575 63.5))
     (stroke (width 0) (type default))
@@
     (stroke (width 0) (type default))
   )
+  (wire (pts (xy 245.11 92.075) (xy 242.57 92.075))
+    (stroke (width 0) (type default))
+  )
   (wire (pts (xy 118.745 80.645) (xy 118.745 81.915))
     (stroke (width 0) (type default))
@@
     (stroke (width 0) (type default))
   )
+  (wire (pts (xy 90.17 165.735) (xy 90.17 167.64))
+    (stroke (width 0) (type default))
+  )
   (wire (pts (xy 103.505 171.45) (xy 103.505 173.99))
     (stroke (width 0) (type default))
@@
     (stroke (width 0) (type default))
   )
+  (wire (pts (xy 242.57 92.075) (xy 242.57 97.155))
+    (stroke (width 0) (type default))
+  )
   (wire (pts (xy 262.89 104.775) (xy 262.89 107.95))
     (stroke (width 0) (type default))
@@
     (stroke (width 0) (type default))
   )
+  (wire (pts (xy 240.665 97.155) (xy 242.57 97.155))
+    (stroke (width 0) (type default))
+  )
   (wire (pts (xy 83.82 73.66) (xy 84.455 73.66))
     (stroke (width 0) (type default))
@@
     (stroke (width 0) (type default))
   )
+  (wire (pts (xy 90.17 186.69) (xy 90.17 188.595))
+    (stroke (width 0) (type default))
+  )
   (wire (pts (xy 158.75 149.225) (xy 158.75 151.765))
     (stroke (width 0) (type default))
@@
     (stroke (width 0) (type default))
   )
+  (wire (pts (xy 86.36 177.165) (xy 90.17 177.165))
+    (stroke (width 0) (type default))
+  )
   (wire (pts (xy 120.015 111.125) (xy 120.015 112.395))
     (stroke (width 0) (type default))
@@
     )
   )
+  (global_label "standby" (shape input) (at 86.36 177.165 180) (fields_autoplaced)
+    (effects (font (size 1.27 1.27)) (justify right))
+    (property "Intersheetrefs" "${INTERSHEET_REFS}" (at 76.0574 177.165 0)
+      (effects (font (size 1.27 1.27)) (justify right) hide)
+    )
+  )
   (global_label "u2" (shape input) (at 233.68 71.755 180) (fields_autoplaced)
     (effects (font (size 1.27 1.27)) (justify right))
@@
     )
   )
+  (global_label "standby" (shape input) (at 240.665 97.155 180) (fields_autoplaced)
+    (effects (font (size 1.27 1.27)) (justify right))
+    (property "Intersheetrefs" "${INTERSHEET_REFS}" (at 230.3624 97.155 0)
+      (effects (font (size 1.27 1.27)) (justify right) hide)
+    )
+  )
   (global_label "bl_ctrl" (shape input) (at 146.685 140.335 180) (fields_autoplaced)
     (effects (font (size 1.27 1.27)) (justify right))
@@
     )
   )
+  (symbol (lib_id "power:GND") (at 90.17 188.595 0) (unit 1)
+    (in_bom yes) (on_board yes) (dnp no) (fields_autoplaced)
+    (property "Reference" "#PWR053" (at 90.17 194.945 0)
+      (effects (font (size 1.27 1.27)) hide)
+    )
+    (property "Value" "GND" (at 90.17 193.04 0)
+      (effects (font (size 1.27 1.27)))
+    )
+    (property "Footprint" "" (at 90.17 188.595 0)
+      (effects (font (size 1.27 1.27)) hide)
+    )
+    (property "Datasheet" "" (at 90.17 188.595 0)
+      (effects (font (size 1.27 1.27)) hide)
+    )
+    (pin "1")
+    (instances
+      (project "ss_v2"
+        (path "/ef461346-06b7-47db-8f2e-cc06c90fb5be"
+          (reference "#PWR053") (unit 1)
+        )
+      )
+    )
+  )
   (symbol (lib_id "power:GND") (at 20.32 43.815 0) (unit 1)
     (in_bom yes) (on_board yes) (dnp no) (fields_autoplaced)
@@
     )
   )
+  (symbol (lib_id "power:+5V") (at 90.17 165.735 0) (unit 1)
+    (in_bom yes) (on_board yes) (dnp no) (fields_autoplaced)
+    (property "Reference" "#PWR054" (at 90.17 169.545 0)
+      (effects (font (size 1.27 1.27)) hide)
+    )
+    (property "Value" "+5V" (at 90.17 160.655 0)
+      (effects (font (size 1.27 1.27)))
+    )
+    (property "Footprint" "" (at 90.17 165.735 0)
+      (effects (font (size 1.27 1.27)) hide)
+    )
+    (property "Datasheet" "" (at 90.17 165.735 0)
+      (effects (font (size 1.27 1.27)) hide)
+    )
+    (pin "1")
+    (instances
+      (project "ss_v2"
+        (path "/ef461346-06b7-47db-8f2e-cc06c90fb5be"
+          (reference "#PWR054") (unit 1)
+        )
+      )
+    )
+  )
   (symbol (lib_id "Device:R") (at 86.36 135.255 0) (unit 1)
     (in_bom yes) (on_board yes) (dnp no) (fields_autoplaced)
@@
     )
   )
+  (symbol (lib_id "Device:R") (at 90.17 182.88 0) (unit 1)
+    (in_bom yes) (on_board yes) (dnp no) (fields_autoplaced)
+    (property "Reference" "R26" (at 92.075 181.61 0)
+      (effects (font (size 1.27 1.27)) (justify left))
+    )
+    (property "Value" "10k" (at 92.075 184.15 0)
+      (effects (font (size 1.27 1.27)) (justify left))
+    )
+    (property "Footprint" "Resistor_SMD:R_1206_3216Metric_Pad1.30x1.75mm_HandSolder" (at 88.392 182.88 90)
+      (effects (font (size 1.27 1.27)) hide)
+    )
+    (property "Datasheet" "~" (at 90.17 182.88 0)
+      (effects (font (size 1.27 1.27)) hide)
+    )
+    (property "Feld4" "" (at 90.17 182.88 0)
+      (effects (font (size 1.27 1.27)) hide)
+    )
+    (pin "1")
+    (pin "2")
+    (instances
+      (project "ss_v2"
+        (path "/ef461346-06b7-47db-8f2e-cc06c90fb5be"
+          (reference "R26") (unit 1)
+        )
+      )
+    )
+  )
   (symbol (lib_id "PJ-313D-B-SMT:PJ-313D-B-SMT") (at 123.19 113.665 180) (unit 1)
     (in_bom yes) (on_board yes) (dnp no)
@@
         )
       )
+    )
+  )
+  (symbol (lib_id "Device:R") (at 90.17 171.45 0) (unit 1)
+    (in_bom yes) (on_board yes) (dnp no) (fields_autoplaced)
+    (property "Reference" "R25" (at 92.075 170.18 0)
+      (effects (font (size 1.27 1.27)) (justify left))
+    )
+    (property "Value" "10k" (at 92.075 172.72 0)
+      (effects (font (size 1.27 1.27)) (justify left))
+    )
+    (property "Footprint" "Resistor_SMD:R_1206_3216Metric_Pad1.30x1.75mm_HandSolder" (at 88.392 171.45 90)
+      (effects (font (size 1.27 1.27)) hide)
+    )
+    (property "Datasheet" "~" (at 90.17 171.45 0)
+      (effects (font (size 1.27 1.27)) hide)
+    )
+    (pin "1")
+    (pin "2")
+    (instances
+      (project "ss_v2"
+        (path "/ef461346-06b7-47db-8f2e-cc06c90fb5be"
+          (reference "R25") (unit 1)
+        )
+      )

Commit message: korrektur der Fehlenden Footprints
Parts:
- J4: footprint (none) -> Connector_IDC:IDC-Header_2x03_P2.54mm_Vertical
- R27: footprint (none) -> Resistor_SMD:R_1206_3216Metric_Pad1.30x1.75mm_HandSolder
Changed lines of the file:
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@@
       (effects (font (size 1.27 1.27)))
     )
-    (property "Footprint" "" (at 43.815 25.4 0)
+    (property "Footprint" "Connector_IDC:IDC-Header_2x03_P2.54mm_Vertical" (at 43.815 25.4 0)
       (effects (font (size 1.27 1.27)) hide)
     )
@@
       (effects (font (size 1.27 1.27)) (justify left))
     )
-    (property "Footprint" "" (at 212.852 75.565 90)
-      (effects (font (size 1.27 1.27)) hide)
-    )
+    (property "Footprint" "Resistor_SMD:R_1206_3216Metric_Pad1.30x1.75mm_HandSolder" (at 212.852 75.565 90)
+      (effects (font (size 1.27 1.27)) hide)
+    )

Commit message: Erster Routing Versuch
Parts:
- removed U3: TPS62125DSG, Package_SON:WSON-8-1EP_2x2mm_P0.5mm_EP0.9x1.6mm_ThermalVias, symbol Regulator_Switching:TPS62125DSG
- added U3: TPS62175DQCR, DQC0010A, symbol TPS62175DQCR:TPS62175DQCR
Connections:
- net +5V: now also U3.10 (VOS), U3.8 (SLEEP)
- net GND: now also U3.1 (PGND), U3.11 (PAD), U3.6 (AGND)
- net VDC: now also U3.2 (VIN), U3.3 (EN)
- net at L1.2: now also U3.9 (SW)
- net at R11.2, R12.1: now also U3.5 (FB)
- net output_power: now reaches J1.2A, J1.2B, Q2.5 (D), Q2.6 (D), Q2.7 (D), Q2.8 (D)
Other:
- moved on the sheet: C6, C7, C8, L1, R11, R12, U4
