File: KiCad/ss_v2/ss_v2-autoroute.kicad_sch (KiCad schematic)
At the start: 62 parts, among them IC1 CH224K, J1 PJ-313D-B-SMT, J3 DC-005-20A, J4 Conn_02x03_Top_Bottom, J5 Conn_02x03_Counter_Clockwise, J6 Conn_01x08_Pin, J7 Conn_01x04, J8 GT-USB-7004, Q1 BSN20, Q2 IRF7416TRPBF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

Commit message: ss_v2 mit neuem Chip umgesetzt. Sieht soweit gut aus, keine Probleme festgestellt. Bitte um Überprüfung.
Parts:
- removed C10, C9: 330p, Resistor_SMD:R_1206_3216Metric_Pad1.30x1.75mm_HandSolder, symbol Device:C
- removed C11, C12: 100n, Resistor_SMD:R_1206_3216Metric_Pad1.30x1.75mm_HandSolder, symbol Device:C
- removed R13, R14: 2k, Resistor_SMD:R_1206_3216Metric_Pad1.30x1.75mm_HandSolder, symbol Device:R
- added F1: 0154003.DR, 0154Series_LTF, symbol 0154003:0154003.DR
Connections:
- net pd-cfg is gone; now on an unnamed net: IC1.9 (CFG3)
- net +12V: no longer Q2.1 (S), Q2.2 (S), Q2.3 (S), Q3.3 (D), R10.2
- net GND: now also C13.2, IC1.2 (CFG1)
- net VDC: now also Q2.1 (S), Q2.2 (S), Q2.3 (S), Q3.3 (D), R10.2, F1.2; no longer J4.2 (Pin_2)
- net scl: no longer names the net of U1.28 (PC5)
- net sda: no longer names the net of U1.27 (PC4)
- new net: F1.1, J4.2 (Pin_2)
- no-connect marks 1 -> 3
