File: KiCad/ss_v2/ss_v2-autoroute.kicad_pcb (KiCad board)
At the start: 2 copper layers, 74.3 x 63 mm, 61 parts, among them IC1 CH224K, J1 PJ-313D-B-SMT, J2 GT-USB-7004, J3 DC-005-20A, J4 Conn_02x03_Top_Bottom, J5 Conn_02x03_Counter_Clockwise, J6 Conn_01x08_Pin, J7 Conn_01x04, Q1 BSN20, Q2 IRF7416TRPBF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

Commit message: GND an 328p gefixt
Routing:
- net GND: track 47.1 -> 51.1 mm, vias 17 -> 19
Changed lines of the file:
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@@
         (effects (font (size 1 1) (thickness 0.15)))
     )
-    (fp_text value "TS-1093C-A15" (at 0 0 unlocked) (layer "F.Fab")
+    (fp_text value "TS-1093C-A15" (at 2.25044 -4.30022 unlocked) (layer "F.Fab")
         (effects (font (size 1 1) (thickness 0.15)))
     )
@@
   (via (at 195.8 94.1) (size 0.8) (drill 0.4) (layers "F.Cu" "B.Cu") (free) (net 1))
   (via (at 232.3 117.5) (size 0.8) (drill 0.4) (layers "F.Cu" "B.Cu") (free) (net 1))
+  (via (at 232.918 104.1146) (size 0.8) (drill 0.4) (layers "F.Cu" "B.Cu") (free) (net 1))
+  (via (at 230.0986 106.8324) (size 0.8) (drill 0.4) (layers "F.Cu" "B.Cu") (free) (net 1))
   (via (at 218.4 116) (size 0.8) (drill 0.4) (layers "F.Cu" "B.Cu") (free) (net 1))
   (via (at 256.025 97.05) (size 0.8) (drill 0.4) (layers "F.Cu" "B.Cu") (free) (net 1))
@@
   (segment (start 256.025 97.05) (end 256.025 94.025) (width 1) (layer "B.Cu") (net 1))
   (segment (start 198.8 92.2) (end 198.8 88.4) (width 1) (layer "B.Cu") (net 1))
+  (segment (start 230.2002 106.8324) (end 232.918 104.1146) (width 1) (layer "B.Cu") (net 1))
+  (segment (start 230.0224 106.8324) (end 230.2002 106.8324) (width 1) (layer "B.Cu") (net 1))
   (segment (start 205.3 115.9) (end 205.3 111.5) (width 1) (layer "B.Cu") (net 1))
   (segment (start 220.975 87.175) (end 221 87.2) (width 1) (layer "B.Cu") (net 1))
